Commit message: camera adjustments

File: gym_panda_reach/envs/base.urdf (robot description, URDF)
Before this commit: robot floor, 1 links, 0 joints
Links:
- link baseLink: geometry collision cylinder length=0.65 radius=0.2; visual cylinder length=0.65 radius=0.2

File: gym_panda_reach/envs/flat_table.urdf (robot description, URDF)
Before this commit: robot cube, 1 links, 0 joints
Links:
- link baseLink: geometry collision box size=0.7 1 0.65; visual box size=0.7 1 0.65
